File: pcb/lul_left/lul_left.kicad_pcb (KiCad board)
At the start: 2 copper layers, 111.5 x 76.8 mm, 54 parts, among them J1 SWD_Ext, J2 Conn_02x04_Odd_Even, SW1 SW_Push, SW10 SW_Push, SW11 SW_Push, SW12 SW_Push, SW13 SW_Push, SW14 SW_Push, SW15 SW_Push, SW16 SW_Push, SW17 SW_Push, SW18 SW_DPDT_x2, SW19 SW_RESET, SW2 SW_Push, SW20 SW_DPDT_x2, SW3 SW_Push, SW4 SW_Push, SW5 SW_Push, SW6 SW_Push, SW7 SW_Push, SW8 SW_Push, SW9 SW_Push, U1 E73-2G4M08S1C, U2 XC6206PxxxMR, U3 DW01A, U4 FS8205, Y1 Crystal_Small

Commit message: switches positioned properly
Parts:
- removed BT1: Battery_Cell, weteor:Coin Cell 2032
- removed C1, C4: 1uF, Capacitor_SMD:C_0603_1608Metric
- removed C2, C3, C5: 0.1uF, Capacitor_SMD:C_0603_1608Metric
- removed D12, D4, D8: D, weteor:D_SOD-123_gold
- removed ENC1: Encoder, weteor:Mitsumi_SIQ-02FVS3
- removed R1, R3: 100R, Resistor_SMD:R_0603_1608Metric
- removed R2: 1k, Resistor_SMD:R_0603_1608Metric
- removed U3: DW01A, Package_TO_SOT_SMD:SOT-23-6
- removed U4: FS8205, Package_TO_SOT_SMD:SOT-23-6
- removed Y1: Crystal_Small, Crystal:Crystal_SMD_3215-2Pin_3.2x1.5mm
- added D18: D, Diode_SMD:D_SOD-123, F.Cu at (106.6, 145.4)
- added D19: D, Diode_SMD:D_SOD-123, F.Cu at (106.6, 148.8)
- added D20: D, Diode_SMD:D_SOD-123, F.Cu at (153.6, 220.1)
- added D21: D, Diode_SMD:D_SOD-123, F.Cu at (153.6, 223.4)
- added D22: D, Diode_SMD:D_SOD-123, F.Cu at (153.6, 226.8)
- added D23: D, Diode_SMD:D_SOD-123, F.Cu at (153.6, 230.1)
- added D24: D, Diode_SMD:D_SOD-123, F.Cu at (153.6, 233.5)
- added D25: D, Diode_SMD:D_SOD-123, F.Cu at (153.6, 236.8)
- added D26: D, Diode_SMD:D_SOD-123, F.Cu at (159.4, 216.7)
- added D27: D, Diode_SMD:D_SOD-123, F.Cu at (159.4, 220.1)
- added D28: D, Diode_SMD:D_SOD-123, F.Cu at (159.4, 223.4)
- added D29: D, Diode_SMD:D_SOD-123, F.Cu at (159.4, 226.8)
- added D30: D, Diode_SMD:D_SOD-123, F.Cu at (159.4, 230.1)
- added D31: D, Diode_SMD:D_SOD-123, F.Cu at (159.4, 233.5)
- added D33: D, Diode_SMD:D_SOD-123, F.Cu at (159.4, 236.8)
- added D34: D, Diode_SMD:D_SOD-123, F.Cu at (165.2, 216.7)
- added D35: D, Diode_SMD:D_SOD-123, F.Cu at (165.2, 220.1)
- added D37: D, Diode_SMD:D_SOD-123, F.Cu at (165.2, 223.4)
- added D38: D, Diode_SMD:D_SOD-123, F.Cu at (165.2, 226.8)
- added D39: D, Diode_SMD:D_SOD-123, F.Cu at (165.2, 230.1)
- added SW21: SW_Push, MX_Only:MXOnly-1U-Hotswap, F.Cu at (174.0, 91.2)
- added SW22: SW_Push, MX_Only:MXOnly-1U-Hotswap, F.Cu at (209.7, 30.3)
- added SW23: SW_Push, MX_Only:MXOnly-1U-Hotswap, F.Cu at (209.6, 49.4)
- added SW24: SW_Push, MX_Only:MXOnly-1U-Hotswap, F.Cu at (209.7, 68.4)
- added SW25: SW_Push, MX_Only:MXOnly-1.75U-Hotswap, F.Cu at (200.2, 91.2)
- added SW26: SW_Push, MX_Only:MXOnly-1U-Hotswap, F.Cu at (228.7, 30.3)
- added SW27: SW_Push, MX_Only:MXOnly-1U-Hotswap, F.Cu at (228.7, 49.4)
- added SW28: SW_Push, MX_Only:MXOnly-1U-Hotswap, F.Cu at (228.7, 68.4)
- added SW29: SW_Push, MX_Only:MXOnly-1U-Hotswap, F.Cu at (247.8, 30.3)
- added SW30: SW_Push, MX_Only:MXOnly-1U-Hotswap, F.Cu at (247.8, 49.4)
- added SW31: SW_Push, MX_Only:MXOnly-1U-Hotswap, F.Cu at (247.8, 68.4)
- added SW32: SW_Push, MX_Only:MXOnly-1U-Hotswap, F.Cu at (266.8, 30.3)
- added SW33: SW_Push, MX_Only:MXOnly-1U-Hotswap, F.Cu at (266.8, 49.4)
- added SW34: SW_Push, MX_Only:MXOnly-1U-Hotswap, F.Cu at (266.8, 68.4)
- added SW_RESET2: SW_RESET, random-keyboard-parts:SKQG-1155865, F.Cu at (172.8, 232.0)
- added SW_RESET_1: SW_RESET, random-keyboard-parts:SKQG-1155865, F.Cu at (96.8, 153.6)
- added SW_SPDT_1: SW_SPDT, Button_Switch_SMD:SW_SPDT_PCM12, F.Cu at (173.0, 218.0)
- added SW_SPDT_2: SW_SPDT, Button_Switch_SMD:SW_SPDT_PCM12, F.Cu at (173.0, 224.9)
- D1, D10, D11, D13, D14, D15, D16, D17, D2, D3, D5, D6, D7, D9: footprint weteor:D_SOD-123_gold -> Diode_SMD:D_SOD-123
- J1: value SWD_Ext -> JST Connector; footprint Connector_PinHeader_2.54mm:PinHeader_1x04_P2.54mm_Vertical -> Connector_JST:JST_PH_S2B-PH-K_1x02_P2.00mm_Horizontal
- J2: value Conn_02x04_Odd_Even -> JST Connector; footprint Connector_PinSocket_1.27mm:PinSocket_2x04_P1.27mm_Vertical -> Connector_JST:JST_PH_S2B-PH-K_1x02_P2.00mm_Horizontal; moved to F.Cu
- SW1, SW10, SW11, SW12, SW14, SW15, SW16, SW17, SW2, SW3, SW4, SW5, SW6, SW7, SW9: footprint weteor:ChocV1_V2_Hotswap -> MX_Only:MXOnly-1U-Hotswap
- SW13: footprint weteor:ChocV1_V2_Hotswap -> MX_Only:MXOnly-1.75U-Hotswap
- SW18, SW20: value SW_DPDT_x2 -> SW_Push; footprint weteor:DPDT - C2837066 -> MX_Only:MXOnly-1U-Hotswap; moved to F.Cu
- SW19: value SW_RESET -> SW_Push; footprint weteor:Micro_Push_Button_3x6x2.5mm -> MX_Only:MXOnly-1U-Hotswap; moved to F.Cu
- SW8: footprint weteor:ChocV1_V2_Hotswap_1.5u -> MX_Only:MXOnly-1U-Hotswap
- U1: value E73-2G4M08S1C -> nice_nano; footprint weteor:E73-2G4M08S1C_bottom -> nice-nano-kicad:nice_nano
- U2: value XC6206PxxxMR -> nice_nano; footprint Package_TO_SOT_SMD:SOT-23 -> nice-nano-kicad:nice_nano
- moved SW4 175.4 mm to (48.3, 29.7), turned to 0 degrees
- moved J1 136.8 mm to (153.6, 240.9), turned to 0 degrees
- moved J2 135.0 mm to (161.6, 240.9), turned to 0 degrees
- moved D16 133.1 mm to (153.6, 216.7), turned to 0 degrees
- moved SW8 130.1 mm to (67.4, 48.8), turned to 0 degrees
- moved U2 117.2 mm to (134.7, 243.8)
- moved U1 115.1 mm to (134.7, 224.6)
- moved D15 101.5 mm to (106.6, 138.7), turned to 0 degrees
- moved SW18 100.1 mm to (190.6, 30.3)
- moved SW7 91.0 mm to (67.3, 29.7), turned to 0 degrees
- moved SW14 89.6 mm to (105.5, 29.7), turned to 0 degrees
- moved D13 87.9 mm to (100.8, 148.8), turned to 0 degrees
- moved SW1 86.8 mm to (29.2, 29.7), turned to 0 degrees
- moved SW2 86.0 mm to (29.2, 48.7), turned to 0 degrees
- moved D6 85.5 mm to (95.0, 148.8), turned to 0 degrees
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Connections:
- D1 pad 1: Row_1 -> Row_1_L
- D10 pad 1: Row_2 -> Row_2_L
- D10 pad 2: Net-(D10-Pad2) -> Net-(D10-A)
- D11 pad 1: Row_3 -> Row_3_L
- D11 pad 2: Net-(D11-Pad2) -> Net-(D11-A)
- D13 pad 1: Row_2 -> Row_1_L
- D13 pad 2: Net-(D13-Pad2) -> Net-(D13-A)
- D14 pad 1: Row_3 -> Row_2_L
- D14 pad 2: Net-(D14-Pad2) -> Net-(D14-A)
- D15 pad 1: Row_1 -> Row_3_L
- D15 pad 2: Net-(D15-Pad2) -> Net-(D15-A)
- D16 pad 1: Row_2 -> Row_4_L
- D16 pad 2: Net-(D16-Pad2) -> Net-(D16-A)
- D17 pad 1: Row_3 -> Row_1_L
- D17 pad 2: Net-(D17-Pad2) -> Net-(D17-A)
- D2 pad 1: Row_2 -> Row_2_L
- D3 pad 1: Row_3 -> Row_3_L
- D5 pad 1: Row_4 -> Row_1_L
- D5 pad 2: Net-(D5-Pad2) -> Net-(D5-A)
- D6 pad 1: Row_1 -> Row_2_L
- D7 pad 1: Row_2 -> Row_3_L
- D9 pad 1: Row_1 -> Row_1_L
- D9 pad 2: Net-(D9-Pad2) -> Net-(D9-A)
- J1 pad 1: GND -> BAT_L
- J1 pad 2: VDD -> GND
- J2 pad 1: GND -> BAT_R
- J2 pad 2: unconnected-(J2-Pad2) -> GND
- SW1 pad 1: Col_1 -> Col_1_L
- SW10 pad 1: Col_3 -> Col_4_L
- SW10 pad 2: Net-(D10-Pad2) -> Net-(D13-A)
- SW11 pad 1: Col_3 -> Col_4_L
- SW11 pad 2: Net-(D11-Pad2) -> Net-(D14-A)
- SW12 pad 1: Col_4 -> Col_4_L
- SW12 pad 2: Net-(D12-Pad2) -> Net-(D15-A)
- SW13 pad 1: Col_4 -> Col_4_L
- SW13 pad 2: Net-(D13-Pad2) -> Net-(D16-A)
- SW14 pad 1: Col_4 -> Col_5
- SW14 pad 2: Net-(D14-Pad2) -> Net-(D17-A)
- SW15 pad 2: Net-(D15-Pad2) -> Net-(D18-A)
- SW16 pad 2: Net-(D16-Pad2) -> Net-(D19-A)
- SW17 pad 2: Net-(D17-Pad2) -> Net-(D20-A)
- SW18 pad 1: +BATT -> Col_1_R
- SW19 pad 1: GND -> Col_1_R
- SW2 pad 1: Col_1 -> Col_1_L
- SW20 pad 1: unconnected-(SW20-Pad1) -> Col_1_R
- SW3 pad 1: Col_1 -> Col_1_L
- SW4 pad 1: Col_5 -> Col_2_L
- SW4 pad 2: Net-(D4-Pad2) -> Net-(D5-A)
- SW5 pad 1: Col_2 -> Col_2_L
- SW6 pad 1: Col_2 -> Col_2_L
- SW7 pad 1: Col_2 -> Col_3_L
- SW7 pad 2: Net-(D8-Pad2) -> Net-(D9-A)
- SW8 pad 1: Col_4 -> Col_3_L
- SW8 pad 2: Net-(D5-Pad2) -> Net-(D10-A)
- SW9 pad 1: Col_3 -> Col_3_L
- SW9 pad 2: Net-(D9-Pad2) -> Net-(D11-A)
- U1 pad 1: Row_4 -> unconnected-(U1-TX0/P0.06-Pad1)
- U1 pad 10: ENC_A -> Col_3_L
- U1 pad 11: Net-(C3-Pad2) -> Col_4_L
- U1 pad 13: Net-(C2-Pad2) -> unconnected-(U1-NFC1/P0.09-Pad13)
- U1 pad 15: unconnected-(U1-Pad15) -> Row_3_L
- U1 pad 17: Row_3 -> Row_1_L
- U1 pad 19: VDD -> unconnected-(U1-AIN5/P0.29-Pad19)
- U1 pad 2: Col_5 -> unconnected-(U1-RX1/P0.08-Pad2)
- U1 pad 21: GND -> VCC
- U1 pad 23: VDD -> GND
- U1 pad 3: Col_4 -> GND
- U1 pad 31: /D+ -> unconnected-(U1-P1.01-Pad31)
- U1 pad 33: Col_2 -> unconnected-(U1-P1.07-Pad33)
- U1 pad 4: Row_1 -> GND
- U1 pad 5: GND -> unconnected-(U1-P0.17-Pad5)
- U1 pad 7: Row_2 -> unconnected-(U1-P0.22-Pad7)
- U1 pad 8: ENC_B -> Col_1_L
- U1 pad 9: ENC_S -> Col_2_L
- U2 pad 1: GND -> unconnected-(U2-TX0/P0.06-Pad1)
- U2 pad 2: VDD -> unconnected-(U2-RX1/P0.08-Pad2)
- U2 pad 3: +BATT -> GND
Routing:
- net GND: track 28.2 -> 0.00 mm, vias 16 -> 0
- net Net-(BT1-Pad2): track 21.0 -> 0.00 mm, vias 1 -> 0
- net Net-(C5-Pad2): track 17.6 -> 0.00 mm, vias 2 -> 0
- net VDD: track 12.9 -> 0.00 mm, vias 9 -> 0
- net Col_4: track 8.72 -> 0.00 mm, vias 6 -> 0
- net Net-(C5-Pad1): track 8.11 -> 0.00 mm, vias 2 -> 0
- net Net-(C2-Pad2): track 7.34 -> 0.00 mm
- net Net-(D23-A): track 6.73 -> 0.00 mm, vias 1 -> 0
- net Net-(U3-Pad1): track 6.61 -> 0.00 mm
- net Net-(U3-Pad3): track 6.43 -> 0.00 mm
- net Net-(C3-Pad2): track 4.84 -> 0.00 mm
- net Net-(R2-Pad2): track 4.66 -> 0.00 mm
- net +BATT: track 4.30 -> 0.00 mm, vias 2 -> 0
- net Net-(D5-Pad2): track 2.77 -> 0.00 mm, vias 1 -> 0
- net Row_4: track 2.25 -> 0.00 mm, vias 1 -> 0
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- added copper zone on B.Cu, net Col_1_L
- added copper zone on F.Cu, net Col_1_L
- added copper zone on B.Cu, net Col_2_L
- added copper zone on F.Cu, net Col_2_L
- added copper zone on B.Cu, net Col_3_L
- added copper zone on F.Cu, net Col_3_L
- added copper zone on B.Cu, net Col_4_L
- added copper zone on F.Cu, net Col_4_L
- added copper zone on B.Cu, net Net-(D10-A)
- added copper zone on B.Cu, net Net-(D11-A)
- added copper zone on B.Cu, net Net-(D13-A)
- added copper zone on B.Cu, net Net-(D14-A)
- added copper zone on B.Cu, net Net-(D15-A)
- added copper zone on B.Cu, net Net-(D16-A)
- added copper zone on B.Cu, net Net-(D17-A)
- added copper zone on B.Cu, net Net-(D5-A)
- added copper zone on B.Cu, net Net-(D9-A)
- added copper zone on B.Cu, net Row_1_L
- added copper zone on F.Cu, net Row_1_L
- added copper zone on B.Cu, net Row_2_L
- added copper zone on F.Cu, net Row_2_L
- added copper zone on B.Cu, net Row_3_L
- added copper zone on F.Cu, net Row_3_L
- removed copper zone on B.Cu, net /D+
- removed copper zone on F.Cu, net /D+
- removed copper zone on B.Cu, net /D-
- removed copper zone on F.Cu, net /D-
- removed copper zone on B.Cu, net Col_1
- removed copper zone on F.Cu, net Col_1
- removed copper zone on B.Cu, net Col_2
- removed copper zone on F.Cu, net Col_2
- removed copper zone on B.Cu, net Col_3
- removed copper zone on F.Cu, net Col_3
- removed copper zone on B.Cu, net Col_4
- removed copper zone on F.Cu, net Col_4
- removed copper zone on B.Cu, net ENC_A
- removed copper zone on F.Cu, net ENC_A
- removed copper zone on B.Cu, net ENC_B
- removed copper zone on F.Cu, net ENC_B
- removed copper zone on B.Cu, net ENC_S
- removed copper zone on F.Cu, net ENC_S
- removed copper zone on B.Cu, net Net-(BT1-Pad2)
- removed copper zone on F.Cu, net Net-(BT1-Pad2)
- removed copper zone on B.Cu, net Net-(D10-Pad2)
- removed copper zone on B.Cu, net Net-(D11-Pad2)
- removed copper zone on B.Cu, net Net-(D12-Pad2)
- removed copper zone on B.Cu, net Net-(D13-Pad2)
- removed copper zone on B.Cu, net Net-(D14-Pad2)
- removed copper zone on B.Cu, net Net-(D15-Pad2)
- removed copper zone on B.Cu, net Net-(D16-Pad2)
- removed copper zone on B.Cu, net Net-(D17-Pad2)
- removed copper zone on F.Cu, net Net-(D21-A)
- removed copper zone on B.Cu, net Net-(D4-Pad2)
- removed copper zone on B.Cu, net Net-(D5-Pad2)
- removed copper zone on B.Cu, net Net-(D8-Pad2)
- removed copper zone on B.Cu, net Net-(D9-Pad2)
- removed copper zone on F.Cu, net Reset
- removed copper zone on B.Cu, net Row_1
- removed copper zone on F.Cu, net Row_1
- removed copper zone on B.Cu, net Row_2
- removed copper zone on F.Cu, net Row_2
- removed copper zone on B.Cu, net Row_3
- removed copper zone on F.Cu, net Row_3
- removed copper zone on B.Cu, net Row_4
- removed copper zone on F.Cu, net Row_4
- removed copper zone on B.Cu, net VBUS
- removed copper zone on F.Cu, net VBUS
- removed copper zone on B.Cu, net VDD
- removed copper zone on F.Cu, net VDD
- removed copper zone on B.Cu, net swclk
- removed copper zone on F.Cu, net swclk
- removed copper zone on B.Cu, net swdio
- removed copper zone on F.Cu, net swdio
Other:
- board size 111.5 x 76.8 mm -> 260 x 84.8 mm
- board text removed: "+"
- board text removed: "-"
- board text removed: "<"
- board text removed: ">"
- board text removed: "c"
- board text removed: "d"
- board text removed: "g"
- board text removed: "on"
- board text removed: "pr"
- board text removed: "v"

Commit message: move components to temporary locations
Parts:
- removed D1, D10, D11, D13, D14, D15, D16, D17, D18, D19, D2, D20, D21, D22, D23, D24, D25, D26, D27, D28, D29, D3, D30, D31, D33, D34, D35, D37, D38, D39, D5, D6, D7, D9: D, Diode_SMD:D_SOD-123
- moved J1 196.1 mm to (25.9, 92.0)
- moved J2 182.4 mm to (253.9, 83.6), turned to 90 degrees
- moved U2 181.8 mm to (233.7, 91.3), turned to 180 degrees
- moved SW_SPDT_1 178.8 mm to (37.2, 101.6)
- moved SW_RESET2 166.3 mm to (273.0, 99.2), turned to 180 degrees
- moved U1 152.6 mm to (61.9, 90.5)
- moved SW_SPDT_2 151.4 mm to (260.4, 101.3)
- moved SW_RESET_1 102.5 mm to (23.8, 81.8)
Connections:
- SW1 pad 1: Col_1_L -> L1
- SW1 pad 2: Net-(D1-A) -> GND
- SW10 pad 1: Col_4_L -> L10
- SW10 pad 2: Net-(D13-A) -> GND
- SW11 pad 1: Col_4_L -> L11
- SW11 pad 2: Net-(D14-A) -> GND
- SW12 pad 1: Col_4_L -> L12
- SW12 pad 2: Net-(D15-A) -> GND
- SW13 pad 1: Col_4_L -> L13
- SW13 pad 2: Net-(D16-A) -> GND
- SW14 pad 1: Col_5 -> L14
- SW14 pad 2: Net-(D17-A) -> GND
- SW15 pad 1: Col_5 -> L15
- SW15 pad 2: Net-(D18-A) -> GND
- SW16 pad 1: Col_5 -> L16
- SW16 pad 2: Net-(D19-A) -> GND
- SW17 pad 1: Col_5 -> L17
- SW17 pad 2: Net-(D20-A) -> GND
- SW2 pad 1: Col_1_L -> L2
- SW2 pad 2: Net-(D2-A) -> GND
- SW3 pad 1: Col_1_L -> L3
- SW3 pad 2: Net-(D3-A) -> GND
- SW4 pad 1: Col_2_L -> L4
- SW4 pad 2: Net-(D5-A) -> GND
- SW5 pad 1: Col_2_L -> L5
- SW5 pad 2: Net-(D6-A) -> GND
- SW6 pad 1: Col_2_L -> L6
- SW6 pad 2: Net-(D7-A) -> GND
- SW7 pad 1: Col_3_L -> L7
- SW7 pad 2: Net-(D9-A) -> GND
- SW8 pad 1: Col_3_L -> L8
- SW8 pad 2: Net-(D10-A) -> GND
- SW9 pad 1: Col_3_L -> L9
- SW9 pad 2: Net-(D11-A) -> GND
- U1 pad 10: Col_3_L -> L6
- U1 pad 11: Col_4_L -> L7
- U1 pad 12: unconnected-(U1-P1.06-Pad12) -> L8
- U1 pad 13: unconnected-(U1-NFC1/P0.09-Pad13) -> L16
- U1 pad 14: Row_4_L -> L15
- U1 pad 15: Row_3_L -> L14
- U1 pad 16: Row_2_L -> L13
- U1 pad 17: Row_1_L -> L12
- U1 pad 18: unconnected-(U1-AIN0/P0.02-Pad18) -> L11
- U1 pad 19: unconnected-(U1-AIN5/P0.29-Pad19) -> L10
- U1 pad 20: unconnected-(U1-AIN7/P0.31-Pad20) -> L9
- U1 pad 31: unconnected-(U1-P1.01-Pad31) -> L17
- U1 pad 5: unconnected-(U1-P0.17-Pad5) -> L1
- U1 pad 6: unconnected-(U1-P0.20-Pad6) -> L2
- U1 pad 7: unconnected-(U1-P0.22-Pad7) -> L3
- U1 pad 8: Col_1_L -> L4
- U1 pad 9: Col_2_L -> L5
- U2 pad 10: Row_3_R -> R14
- U2 pad 11: Row_4_R -> R15
- U2 pad 12: unconnected-(U2-P1.06-Pad12) -> R16
- U2 pad 13: unconnected-(U2-NFC1/P0.09-Pad13) -> R8
- U2 pad 14: Col_4_R -> R7
- U2 pad 15: Col_3_R -> R6
- U2 pad 16: Col_2_R -> R5
- U2 pad 17: Col_1_R -> R4
- U2 pad 18: unconnected-(U2-AIN0/P0.02-Pad18) -> R3
- U2 pad 19: unconnected-(U2-AIN5/P0.29-Pad19) -> R2
- U2 pad 20: unconnected-(U2-AIN7/P0.31-Pad20) -> R1
- U2 pad 33: unconnected-(U2-P1.07-Pad33) -> R17
- U2 pad 5: unconnected-(U2-P0.17-Pad5) -> R9
- U2 pad 6: unconnected-(U2-P0.20-Pad6) -> R10
- U2 pad 7: unconnected-(U2-P0.22-Pad7) -> R11
- U2 pad 8: Row_1_R -> R12
- U2 pad 9: Row_2_R -> R13
Routing:
- added copper zone on B.Cu, net L12
- added copper zone on F.Cu, net L12
- added copper zone on B.Cu, net L13
- added copper zone on F.Cu, net L13
- added copper zone on B.Cu, net L14
- added copper zone on F.Cu, net L14
- added copper zone on B.Cu, net L17
- added copper zone on F.Cu, net L17
- added copper zone on B.Cu, net L4
- added copper zone on F.Cu, net L4
- added copper zone on B.Cu, net L5
- added copper zone on F.Cu, net L5
- added copper zone on B.Cu, net L6
- added copper zone on F.Cu, net L6
- added copper zone on B.Cu, net L7
- added copper zone on F.Cu, net L7
- removed copper zone on B.Cu, net Col_1_L
- removed copper zone on F.Cu, net Col_1_L
- removed copper zone on B.Cu, net Col_2_L
- removed copper zone on F.Cu, net Col_2_L
- removed copper zone on B.Cu, net Col_3_L
- removed copper zone on F.Cu, net Col_3_L
- removed copper zone on B.Cu, net Col_4_L
- removed copper zone on F.Cu, net Col_4_L
- removed copper zone on B.Cu, net Col_5
- removed copper zone on F.Cu, net Col_5
- removed copper zone on B.Cu, net Net-(D1-A)
- removed copper zone on B.Cu, net Net-(D10-A)
- removed copper zone on B.Cu, net Net-(D11-A)
- removed copper zone on B.Cu, net Net-(D13-A)
- removed copper zone on B.Cu, net Net-(D14-A)
- removed copper zone on B.Cu, net Net-(D15-A)
- removed copper zone on B.Cu, net Net-(D16-A)
- removed copper zone on B.Cu, net Net-(D17-A)
- removed copper zone on B.Cu, net Net-(D2-A)
- removed copper zone on B.Cu, net Net-(D3-A)
- removed copper zone on B.Cu, net Net-(D5-A)
- removed copper zone on B.Cu, net Net-(D6-A)
- removed copper zone on B.Cu, net Net-(D7-A)
- removed copper zone on B.Cu, net Net-(D9-A)
- removed copper zone on B.Cu, net Row_1_L
- removed copper zone on F.Cu, net Row_1_L
- removed copper zone on B.Cu, net Row_2_L
- removed copper zone on F.Cu, net Row_2_L
- removed copper zone on B.Cu, net Row_3_L
- removed copper zone on F.Cu, net Row_3_L

Commit message: move components, add dimension labels, add breakable tabs between pcb bodies
Parts:
- added REF**: Hole_Breakaway-Tabs, zzkeeb:Hole_Breakaway-Tabs, F.Cu at (139.4, 59.5)
- added REF**: Hole_Breakaway-Tabs, zzkeeb:Hole_Breakaway-Tabs, F.Cu at (144.8, 25.9)
- added REF**: Hole_Breakaway-Tabs, zzkeeb:Hole_Breakaway-Tabs, F.Cu at (139.4, 102.5)
- added REF**: Hole_Breakaway-Tabs, zzkeeb:Hole_Breakaway-Tabs, F.Cu at (139.4, 25.9)
- added REF**: Hole_Breakaway-Tabs, zzkeeb:Hole_Breakaway-Tabs, F.Cu at (144.8, 59.5)
- added REF**: Hole_Breakaway-Tabs, zzkeeb:Hole_Breakaway-Tabs, F.Cu at (144.8, 102.5)
- SW21: footprint MX_Only:MXOnly-1U-Hotswap -> MX_Only:MXOnly-1.75U-Hotswap
- SW25: footprint MX_Only:MXOnly-1.75U-Hotswap -> MX_Only:MXOnly-1U-Hotswap
- moved SW_RESET2 239.7 mm to (34.1, 79.5)
- moved SW_RESET_1 226.3 mm to (250.1, 79.5)
- moved SW25 165.4 mm to (34.8, 94.3)
- moved SW_SPDT_2 141.3 mm to (119.1, 104.1)
- moved U2 139.7 mm to (94.0, 94.3)
- moved SW22 138.9 mm to (70.8, 33.2)
- moved SW24 138.9 mm to (70.8, 71.3)
- moved SW26 138.9 mm to (89.9, 33.2)
- moved SW28 138.9 mm to (89.9, 71.3)
- moved SW29 138.9 mm to (108.9, 33.2)
- moved SW31 138.9 mm to (108.9, 71.3)
- moved SW32 138.9 mm to (128.0, 33.2)
- moved SW18 138.9 mm to (51.8, 33.2)
- moved SW19 138.9 mm to (51.8, 52.2)
- moved SW20 138.9 mm to (51.8, 71.3)
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Connections:
- SW18 pad 1: Col_1_R -> R1
- SW18 pad 2: Net-(D21-A) -> GND
- SW19 pad 1: Col_1_R -> R2
- SW19 pad 2: Net-(D22-A) -> GND
- SW20 pad 1: Col_1_R -> R3
- SW20 pad 2: Net-(D23-A) -> GND
- SW21 pad 1: Col_1_R -> R4
- SW21 pad 2: Net-(D24-A) -> GND
- SW22 pad 1: Col_2_R -> R5
- SW22 pad 2: Net-(D25-A) -> GND
- SW23 pad 1: Col_2_R -> R6
- SW23 pad 2: Net-(D26-A) -> GND
- SW24 pad 1: Col_2_R -> R7
- SW24 pad 2: Net-(D27-A) -> GND
- SW25 pad 1: Col_2_R -> R8
- SW25 pad 2: Net-(D28-A) -> GND
- SW26 pad 1: Col_3_R -> R9
- SW26 pad 2: Net-(D29-A) -> GND
- SW27 pad 1: Col_3_R -> R10
- SW27 pad 2: Net-(D30-A) -> GND
- SW28 pad 1: Col_3_R -> R11
- SW28 pad 2: Net-(D31-A) -> GND
- SW29 pad 1: Col_4_R -> R12
- SW29 pad 2: Net-(D33-A) -> GND
- SW30 pad 1: Col_4_R -> R13
- SW30 pad 2: Net-(D34-A) -> GND
- SW31 pad 1: Col_4_R -> R14
- SW31 pad 2: Net-(D35-A) -> GND
- SW32 pad 1: Col_5_R -> R15
- SW32 pad 2: Net-(D37-A) -> GND
- SW33 pad 1: Col_5_R -> R16
- SW33 pad 2: Net-(D38-A) -> GND
- SW34 pad 1: Col_5_R -> R17
- SW34 pad 2: Net-(D39-A) -> GND
- U1 pad 1: unconnected-(U1-TX0/P0.06-Pad1) -> L1
- U1 pad 10: L6 -> L7
- U1 pad 11: L7 -> L8
- U1 pad 12: L8 -> L9
- U1 pad 13: L16 -> L17
- U1 pad 14: L15 -> L16
- U1 pad 15: L14 -> L15
- U1 pad 16: L13 -> L14
- U1 pad 17: L12 -> L13
- U1 pad 18: L11 -> L12
- U1 pad 19: L10 -> L11
- U1 pad 20: L9 -> L10
- U1 pad 31: L17 -> unconnected-(U1-P1.01-Pad31)
- U1 pad 5: L1 -> L2
- U1 pad 6: L2 -> L3
- U1 pad 7: L3 -> L4
- U1 pad 8: L4 -> L5
- U1 pad 9: L5 -> L6
- U2 pad 1: unconnected-(U2-TX0/P0.06-Pad1) -> R9
- U2 pad 10: R14 -> R15
- U2 pad 11: R15 -> R16
- U2 pad 12: R16 -> R17
- U2 pad 33: R17 -> unconnected-(U2-P1.07-Pad33)
- U2 pad 5: R9 -> R10
- U2 pad 6: R10 -> R11
- U2 pad 7: R11 -> R12
- U2 pad 8: R12 -> R13
- U2 pad 9: R13 -> R14
Other:
- board size 260 x 84.8 mm -> 238.5 x 84.2 mm
- board text added: "LEFT"
- board text added: "RIGHT"
