File: pcb/lul_left/lul_left.kicad_pcb (KiCad board)
At the start: 2 copper layers, 238.5 x 84.2 mm, 48 parts, among them J1 JST Connector, J2 JST Connector, SW1 SW_Push, SW10 SW_Push, SW11 SW_Push, SW12 SW_Push, SW13 SW_Push, SW14 SW_Push, SW15 SW_Push, SW16 SW_Push, SW17 SW_Push, SW18 SW_Push, SW19 SW_Push, SW2 SW_Push, SW20 SW_Push, SW21 SW_Push, SW22 SW_Push, SW23 SW_Push, SW24 SW_Push, SW25 SW_Push, SW26 SW_Push, SW27 SW_Push, SW28 SW_Push, SW29 SW_Push, SW3 SW_Push, SW30 SW_Push, SW31 SW_Push, SW32 SW_Push, SW33 SW_Push, SW34 SW_Push, SW4 SW_Push, SW5 SW_Push, SW6 SW_Push, SW7 SW_Push, SW8 SW_Push, SW9 SW_Push, U1 nice_nano, U2 nice_nano

Commit message: add full grounded copper fills to top and bottom layers
Routing:
- added copper zone on B.Cu, net GND
- added copper zone on F.Cu, net GND
Changed lines of the file:
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@@
   (segment (start 74.050635 80.645) (end 44.219792 80.645) (width 0.254) (layer "B.Cu") (net 53))
   (segment (start 41.149 77.574208) (end 41.148999 62.988792) (width 0.254) (layer "B.Cu") (net 53))
+  (zone (net 1) (net_name "GND") (layers "F&B.Cu") (hatch edge 0.5)
+    (priority 2)
+    (connect_pads (clearance 0.254))
+    (min_thickness 0.254) (filled_areas_thickness no)
+    (fill yes (thermal_gap 0.5) (thermal_bridge_width 0.5))
+    (polygon
+      (pts
+        (xy 19.47 109.588)
+        (xy 19.47 19.037)
+        (xy 142.152 18.783)
+        (xy 264.58 18.91)
+        (xy 264.58 109.588)
+        (xy 142.152 109.588)
+      )
+    )
+  )
   (zone (net 33) (net_name "L14") (layer "B.Cu") (hatch edge 0.508)
     (priority 1)
