File: pcb/lul_left/lul_left.kicad_pcb (KiCad board)
At the start: 2 copper layers, 238.5 x 84.2 mm, 48 parts, among them J1 JST Connector, J2 JST Connector, SW1 SW_Push, SW10 SW_Push, SW11 SW_Push, SW12 SW_Push, SW13 SW_Push, SW14 SW_Push, SW15 SW_Push, SW16 SW_Push, SW17 SW_Push, SW18 SW_Push, SW19 SW_Push, SW2 SW_Push, SW20 SW_Push, SW21 SW_Push, SW22 SW_Push, SW23 SW_Push, SW24 SW_Push, SW25 SW_Push, SW26 SW_Push, SW27 SW_Push, SW28 SW_Push, SW29 SW_Push, SW3 SW_Push, SW30 SW_Push, SW31 SW_Push, SW32 SW_Push, SW33 SW_Push, SW34 SW_Push, SW4 SW_Push, SW5 SW_Push, SW6 SW_Push, SW7 SW_Push, SW8 SW_Push, SW9 SW_Push, U1 nice_nano, U2 nice_nano

Commit message: fix small connection issue
Connections:
- U2 pad 7: R16 -> R14
- U2 pad 8: R6 -> R17
Changed lines of the file:
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@@
       (net 47 "R11") (pinfunction "P0.20") (pintype "input"))
     (pad "7" thru_hole circle (at 1.27 7.62 180) (size 1.7526 1.7526) (drill 1.0922) (layers "*.Cu" "*.SilkS" "*.Mask")
-      (net 52 "R16") (pinfunction "P0.22") (pintype "input"))
+      (net 50 "R14") (pinfunction "P0.22") (pintype "input"))
     (pad "8" thru_hole circle (at 3.81 7.62 180) (size 1.7526 1.7526) (drill 1.0922) (layers "*.Cu" "*.SilkS" "*.Mask")
-      (net 42 "R6") (pinfunction "P0.24") (pintype "input"))
+      (net 53 "R17") (pinfunction "P0.24") (pintype "input"))
     (pad "9" thru_hole circle (at 6.35 7.62 180) (size 1.7526 1.7526) (drill 1.0922) (layers "*.Cu" "*.SilkS" "*.Mask")
       (net 52 "R16") (pinfunction "P1.00") (pintype "input"))

Commit message: edge cuts fixed
Parts:
- added G***: LOGO, LOGO, F.Cu at (249.6, 75.6)
- added G***: LOGO, LOGO, F.Cu at (33.4, 78.7)
Routing:
- net L7: track 172.0 -> 173.4 mm
- net L4: track 191.2 -> 189.8 mm
- net GND: vias 22 -> 0
Other:
- outline, holes or cut-outs redrawn

Commit message: fix footprint courtyard error in MX_1U and MX_1.75U
Parts:
- renumbered G*** to G1, G*** to G2
